Commit message: Add files via upload

File: arduinobot_description/urdf/arduinobot.urdf.xacro (robot description, xacro)
@@ -1,10 +1,6 @@
 <?xml version="1.0"?>
 <robot xmlns:xacro="http://www.ros.org/wiki/xacro" name="arduinobot">
-    <!-- Include Gazebo Parameters -->
-    <xacro:include filename="$(find arduinobot_description)/urdf/arduinobot_gazebo.xacro" />
-    <!-- Include ros2_control Plugins -->
-    <xacro:include filename="$(find arduinobot_description)/urdf/arduinobot_ros2_control.xacro" />
     <!-- Useful XACRO Variables (Properties) -->
-    <xacro:property name="PI" value="3.14159265359" />
+    <xacro:property name="PI" value="3.14" />
     <xacro:property name="effort" value="30.0" />
     <xacro:property name="velocity" value="10.0" />
@@ -23,5 +19,5 @@
             <plugin>transmission_interface/SimpleTransmission</plugin>
             <actuator name="motor_${number}" role="actuator1"/>
-            <joint name="joint_${number}"    role="joint1">
+            <joint name="joint_${number}" role="joint1">
                 <mechanical_reduction>1.0</mechanical_reduction>
             </joint>
@@ -63,5 +59,5 @@
         <xacro:default_inertial mass="0.1"/>
         <visual>
-            <origin rpy=" 0 -${PI / 2} ${PI / 2}" xyz="0.19 0.06 -0.08"/>
+            <origin rpy="0 -${PI / 2} ${PI / 2}" xyz="0.19 0.06 -0.08"/>
             <geometry>
                 <mesh filename="package://arduinobot_description/meshes/forward_drive_arm.STL" scale="0.01 0.01 0.01"/>
@@ -69,5 +65,5 @@
         </visual>
         <collision>
-            <origin rpy=" 0 -${PI / 2} ${PI / 2}" xyz="0.19 0.06 -0.08"/>
+            <origin rpy="0 -${PI / 2} ${PI / 2}" xyz="0.19 0.06 -0.08"/>
             <geometry>
                 <mesh filename="package://arduinobot_description/meshes/forward_drive_arm.STL" scale="0.01 0.01 0.01"/>
@@ -141,54 +137,113 @@
         <origin xyz="0 0 0" rpy="0 0 0"/>
     </joint>
-    <joint name ="joint_1" type="revolute">
+    <joint name="joint_1" type="revolute">
         <parent link="base_link"/>
-        <child link = "base_plate"/>
-        <origin xyz="0 0 0.307"/>
+        <child link="base_plate"/>
+        <origin xyz="0 0 0.307" />
         <axis xyz="0 0 1"/>
-        <limit lower="-${PI / 2}" upper="${PI / 2}"
-               effort="${effort}" velocity="${velocity}"/>
-    </joint>
-    <joint name ="joint_2" type="revolute">
+        <limit lower="-${PI / 2}" upper="${PI / 2}" effort="${effort}" velocity="${velocity}"/>
+    </joint>
+    <joint name="joint_2" type="revolute">
         <parent link="base_plate"/>
-        <child link = "forward_drive_arm"/>
+        <child link="forward_drive_arm"/>
         <origin xyz="-0.02 0 0.35"/>
         <axis xyz="1 0 0"/>
-        <limit lower="-${PI / 2}" upper="${PI / 2}"
-                effort="${effort}" velocity="${velocity}"/>
-    </joint>
-    <joint name ="joint_3" type="revolute">
+        <limit lower="-${PI / 2}" upper="${PI / 2}" effort="${effort}" velocity="${velocity}"/>
+    </joint>
+    <joint name="joint_3" type="revolute">
         <parent link="forward_drive_arm"/>
-        <child link = "horizontal_arm"/>
+        <child link="horizontal_arm"/>
         <origin xyz="0 0 0.8"/>
         <axis xyz="1 0 0"/>
-        <limit lower="-${PI / 2}" upper="${PI / 2}"
-               effort="${effort}" velocity="${velocity}"/>
-    </joint>
-    <joint name ="horizontal_arm_to_claw_support" type="fixed">
+        <limit lower="-${PI / 2}" upper="${PI / 2}" effort="${effort}" velocity="${velocity}"/>
+    </joint>
+    <joint name="horizontal_arm_to_claw_support" type="fixed">
         <parent link="horizontal_arm"/>
-        <child link = "claw_support"/>
+        <child link="claw_support"/>
         <origin xyz="0 0.82 0"/>
     </joint>
-    <joint name ="joint_4" type="revolute">
+    <joint name="joint_4" type="revolute">
         <parent link="claw_support"/>
-        <child link = "gripper_right"/>
+        <child link="gripper_right"/>
         <origin xyz="-0.04 0.13 -0.1"/>
         <axis xyz="0 0 1"/>
-        <limit lower="-${PI / 2}" upper="0.0"
-               effort="${effort}" velocity="${velocity}"/>
-    </joint>
-    <joint name ="joint_5" type="revolute">
+        <limit lower="-${PI / 2}" upper="0.0" effort="${effort}" velocity="${velocity}"/>
+    </joint>
+    <joint name="joint_5" type="revolute">
         <parent link="claw_support"/>
-        <child link = "gripper_left"/>
+        <child link="gripper_left"/>
         <origin xyz="-0.22 0.13 -0.1"/>
         <axis xyz="0 0 1"/>
-        <limit lower="0.0" upper="${PI / 2}"
-               effort="${effort}" velocity="${velocity}"/>
+        <limit lower="0.0" upper="${PI / 2}" effort="${effort}" velocity="${velocity}"/>
         <mimic joint="joint_4" multiplier="-1"/>
     </joint>
-    <!-- Transmissions-->
-    <xacro:default_transmission number="1"/>
-    <xacro:default_transmission number="2"/>
-    <xacro:default_transmission number="3"/>
-    <xacro:default_transmission number="4"/>
+    <!-- Transmissions -->
+    <transmission name="trans_joint_1">
+        <type>transmission_interface/SimpleTransmission</type>
+        <joint name="joint_1">
+            <hardwareInterface>hardware_interface/PositionJointInterface</hardwareInterface>
+        </joint>
+        <actuator name="motor_joint_1">
+            <hardwareInterface>hardware_interface/PositionJointInterface</hardwareInterface>
+        </actuator>
+    </transmission>
+    <transmission name="trans_joint_2">
+        <type>transmission_interface/SimpleTransmission</type>
+        <joint name="joint_2">
+            <hardwareInterface>hardware_interface/PositionJointInterface</hardwareInterface>
+        </joint>
+        <actuator name="motor_joint_2">
+            <hardwareInterface>hardware_interface/PositionJointInterface</hardwareInterface>
+        </actuator>
+    </transmission>
+    <transmission name="trans_joint_3">
+        <type>transmission_interface/SimpleTransmission</type>
+        <joint name="joint_3">
+            <hardwareInterface>hardware_interface/PositionJointInterface</hardwareInterface>
+        </joint>
+        <actuator name="motor_joint_3">
+            <hardwareInterface>hardware_interface/PositionJointInterface</hardwareInterface>
+        </actuator>
+    </transmission>
+    <transmission name="trans_joint_4">
+        <type>transmission_interface/SimpleTransmission</type>
+        <joint name="joint_4">
+            <hardwareInterface>hardware_interface/PositionJointInterface</hardwareInterface>
+        </joint>
+        <actuator name="motor_joint_4">
+            <hardwareInterface>hardware_interface/PositionJointInterface</hardwareInterface>
+        </actuator>
+    </transmission>
+    <!-- ros2_control hardware definition -->
+    <ros2_control name="RobotSystem" type="system">
+        <hardware>
+            <plugin>gazebo_ros2_control/GazeboSystem</plugin>
+        </hardware>
+        <joint name="joint_1">
+            <command_interface name="position"/>
+            <state_interface name="position"/>
+        </joint>
+        <joint name="joint_2">
+            <command_interface name="position"/>
+            <state_interface name="position"/>
+        </joint>
+        <joint name="joint_3">
+            <command_interface name="position"/>
+            <state_interface name="position"/>
+        </joint>
+        <joint name="joint_4">
+            <command_interface name="position"/>
+            <command_interface name="velocity"/>
+            <state_interface name="position"/>
+            <state_interface name="velocity"/>
+        </joint>
+    </ros2_control>
+    <!-- Gazebo ros2_control plugin -->
+    <gazebo>
+        <plugin filename="libgazebo_ros2_control.so" name="gazebo_ros2_control">
+            <robot_param>robot_description</robot_param>
+            <robot_param_node>robot_state_publisher</robot_param_node>
+            <parameters>$(find arduinobot_controller)/config/arduinobot_controllers.yaml</parameters>
+        </plugin>
+    </gazebo>
 </robot>

File: arduinobot_description/urdf/arduinobot_ros2_control.xacro (robot description, xacro)
@@ -1,46 +1,24 @@
 <?xml version="1.0"?>
 <robot xmlns:xacro="http://www.ros.org/wiki/xacro" name="arduinobot">
-    <ros2_control name="RobotSystem" type="system">
-        <xacro:property name="PI" value="3.14159265359" />
-        <!-- ros2_control Gazebo -->
-        <hardware>
-            <plugin>gazebo_ros2_control/GazeboSystem</plugin>
-        </hardware>
-        <joint name="joint_1">
-            <command_interface name="position">
-            <param name="min">-${PI / 2}</param>
-            <param name="max">${PI / 2}</param>
-            </command_interface>
-            <state_interface name="position"/>
-        </joint>
-        <joint name="joint_2">
-            <command_interface name="position">
-            <param name="min">-${PI / 2}</param>
-            <param name="max">${PI / 2}</param>
-            </command_interface>
-            <state_interface name="position"/>
-        </joint>
-        <joint name="joint_3">
-            <command_interface name="position">
-            <param name="min">-${PI / 2}</param>
-            <param name="max">${PI / 2}</param>
-            </command_interface>
-            <state_interface name="position"/>
-        </joint>
-        <joint name="joint_4">
-            <command_interface name="position">
-            <param name="min">-${PI / 2}</param>
-            <param name="max">0.0</param>
-            </command_interface>
-            <state_interface name="position"/>
-        </joint>
-        <joint name="joint_5">
-            <param name="mimic">joint_4</param>
-            <param name="multiplier">-1</param>
-            <command_interface name="position">
-            <param name="min">0.0</param>
-            <param name="max">${PI / 2}</param>
-            </command_interface>
-        </joint>
-    </ros2_control>
+  <ros2_control name="RobotSystem" type="system">
+    <hardware>
+      <plugin>gazebo_ros2_control/GazeboSystem</plugin>
+    </hardware>
+    <joint name="joint_1">
+      <command_interface name="position"/>
+      <state_interface name="position"/>
+    </joint>
+    <joint name="joint_2">
+      <command_interface name="position"/>
+      <state_interface name="position"/>
+    </joint>
+    <joint name="joint_3">
+      <command_interface name="position"/>
+      <state_interface name="position"/>
+    </joint>
+    <joint name="joint_4">
+      <command_interface name="position"/>
+      <state_interface name="position"/>
+    </joint>
+  </ros2_control>
 </robot>
